File: Node V10/Node V10.kicad_pcb (KiCad board)
At the start: 2 copper layers, 12 parts, among them J1 Soil Sensor - 1, J2 Soil Sensor - 2, J3 Soil Sensor - 3, J4 Soil Sensor - 4, J5 PiicoDev, J6 Xiao Battery Connectors, U1 MCU, U2 Nano Power Timer

Commit message: Ready for fab (flip to front)
Parts:
- added REF**: MountingHole_4mm, MountingHole:MountingHole_4mm, F.Cu at (124.5, 98.4)
- added REF**: MountingHole_4mm, MountingHole:MountingHole_4mm, F.Cu at (209.5, 58.4)
- moved U2 103.4 mm to (171.8, 98.4), turned to 90 degrees
- moved J6 89.5 mm to (165.3, 69.1), turned to 90 degrees
- moved TP1 69.0 mm to (165.1, 97.5), turned to -90 degrees
- moved J3 57.7 mm to (147.3, 86.4), turned to 0 degrees
- moved R2 54.6 mm to (165.1, 87.4), turned to -90 degrees
- moved J1 52.9 mm to (132.1, 86.4), turned to 0 degrees
- moved J2 52.8 mm to (137.2, 86.4), turned to 0 degrees
- moved J4 50.9 mm to (142.2, 86.4), turned to 0 degrees
- moved R1 39.2 mm to (165.1, 76.5), turned to -90 degrees
- moved TP2 35.9 mm to (165.1, 74.2), turned to -90 degrees
- moved U1 25.4 mm to (129.6, 58.5)
- moved J5 20.4 mm to (162.3, 71.4), turned to 180 degrees
- renumbered GND to TP1, Vbatt to TP2
Connections:
- U1 pad 10: /SCL -> +3V3
- U1 pad 11: /SDA -> /SCL
- U1 pad 12: /Done -> /SDA
- U1 pad 13: (no net) -> /Done
- U1 pad 14: (no net) -> unconnected-(U1-GP44-Pad14)
- U1 pad 8: GND -> unconnected-(U1-5V-Pad8)
- U1 pad 9: +3V3 -> GND
Routing:
- net +3V3: track 0.00 -> 47.3 mm
- net +BATT: track 0.00 -> 39.5 mm
- net /Soil_Sensor_1: track 0.00 -> 34.1 mm
- net /Done: track 0.00 -> 32.0 mm
- net /Soil_Sensor_2: track 0.00 -> 31.6 mm
- net /Soil_Sensor_3: track 0.00 -> 26.5 mm
- net /Soil_Sensor_4: track 0.00 -> 21.8 mm
- net /SCL: track 0.00 -> 16.0 mm
- net /SDA: track 0.00 -> 12.4 mm
- net /Vbatt_sense: track 0.00 -> 3.30 mm
- net GND: track 0.00 -> 2.54 mm
- added copper zone on B.Cu, net GND
Other:
- board outline added: 93 x 48 mm

Commit message: Updates
Parts:
- J1, J2, J3, J4, J5, J6, R1, R2, REF** (x2), TP1, TP2, U1, U2: moved to B.Cu
- moved REF** 75.8 mm to (133.7, 58.4), turned to 180 degrees
- moved REF** 67.2 mm to (191.7, 98.4), turned to 180 degrees
- moved U1 56.9 mm to (186.5, 58.5), turned to 180 degrees
- moved J1 52.0 mm to (184.1, 86.4), turned to 180 degrees
- moved J2 41.8 mm to (179.0, 86.4), turned to 180 degrees
- moved J4 31.7 mm to (173.9, 86.4), turned to 180 degrees
- moved U2 27.6 mm to (144.3, 98.4)
- moved J3 21.5 mm to (168.8, 86.4), turned to 180 degrees
- moved J6 14.6 mm to (150.8, 69.1)
- moved R1 14.1 mm to (151.0, 76.5)
- moved R2 14.1 mm to (151.0, 87.4)
- moved TP1 14.1 mm to (151.0, 97.5)
- moved TP2 14.1 mm to (151.0, 74.2)
- moved J5 8.48 mm to (153.8, 71.4), turned to 0 degrees
Routing:
- added copper zone on F.Cu, net GND
- removed copper zone on B.Cu, net GND
Other:
- board size 93 x 48 mm -> 66 x 48 mm
